File: Projeto Euler 2022.brd (EAGLE design)
At the start: 395.7 x 237.4 mm, 33 parts, among them M1 MOTOR_HDR, U1 ARDUINO-UNO-R3-SHIELD, U2 LCD-16X2JHD-162A

Commit message: Atualização do projeto.
Parts:
- removed BAT1: 9V, Tinkercad:BATTERY-GENERIC
- removed D1, D4: RED, Tinkercad:LEDRD254W60D565H860B
- removed D3: LED-RGBRCBG-PTH, Tinkercad:LED-RGB-5MM
- removed D5: BLUE, Tinkercad:LEDRD254W60D565H860B_B
- removed D6: GREEN, Tinkercad:LEDRD254W60D565H860B_G
- removed R10, R11, R12, R4: 480, Tinkercad:RESAD1016W63L850D250B
- removed R5: 2000, Tinkercad:RESAD1016W63L850D250B
- removed R6: 330, Tinkercad:RESAD1016W63L850D250B
- removed R7: 620, Tinkercad:RESAD1016W63L850D250B
- removed R8: 1000, Tinkercad:RESAD1016W63L850D250B
- removed R9: 3300, Tinkercad:RESAD1016W63L850D250B
- removed S10, S3, S4, S5, S6, S7, S8, S9: SWITCH_MOMENTARY, Tinkercad:SWITCH-MOMENTARY-PTH-6.5MM
- removed S2: TOGGLE, Tinkercad:SWITCH-SPDT-PTH-8.5X3.7MM
- added R13, R14, R15: 10k, Tinkercad:RESAD1016W63L850D250B
- added S11, S12, S13: SWITCH_MOMENTARY, Tinkercad:SWITCH-MOMENTARY-PTH-6.5MM
- R3: value 150 -> 10
- moved R2 107.0 mm to (194.1, 84.8), turned to 270 degrees
- moved R1 68.1 mm to (60.9, 133.5)
- moved S1 68.1 mm to (63.4, 150.0)
- moved M1 53.7 mm to (8.26, 139.3)
- moved U1 42.9 mm to (90.5, 69.6)
- moved D2 42.9 mm to (54.5, 146.2)
- moved R3 42.9 mm to (55.8, 141.1)
- moved RPOT1 42.9 mm to (153.4, 64.4)
- moved U2 42.9 mm to (175.0, 36.6)
Connections:
- removed net D1_A: D1.1, R2.1
- removed net D3_C: D3.C, R12.2
- removed net D4_A: D4.1, R4.2
- removed net D5_A: D5.1, R10.2
- removed net D6_A: D6.1, R11.2
- removed net S10_3: D3.G, R11.1, S10.3, S10.4
- removed net S8_3: D3.R, R4.1, S8.3, S8.4
- removed net S9_3: D3.B, R10.1, S9.3, S9.4
- new net U1_D10: R13.2, S11.1, S11.2, U1.D10
- new net U1_D11: R1.2, S1.1, S1.2, U1.D11
- new net U1_D9: R14.2, S12.1, S12.2, U1.D9
- new net U2_LED+: R2.2, U2.15
- net U1_5V: now also R2.1, S11.3, S11.4, S12.3, S12.4, S13.3, S13.4; no longer R5.1, S10.1, S8.1, S9.1
- net U1_D8: now also R15.2, S13.1, S13.2; no longer R1.2, S1.1, S1.2
- net U1_GND: now also R13.1, R14.1, R15.1; no longer D4.2, D5.2, D6.2, R12.1, R5.2, R6.1, R6.2, R7.1, R7.2, R8.1, R8.2, R9.1, R9.2, S3.1, S3.2, S3.3, S3.4, S4.1, S4.2, S4.3, S4.4, S5.1, S5.2, S5.3, S5.4, S6.1, S6.2, S6.3, S6.4, S7.1, S7.2, S7.3, S7.4
Other:
- board size 395.7 x 237.4 mm -> 230.6 x 157.4 mm
